File: ADCS/ADCS.kicad_pcb (KiCad board)
At the start: 2 copper layers, 84 x 84 mm, 85 parts, among them J1 Conn_01x02, J10 Conn_01x04, J11 Conn_01x03, J12 Conn_01x08, J14 Conn_01x02, J15 Conn_01x02, J16 SWD_TagConnect, J2 Conn_01x02, J3 Conn_01x02, J4 Conn_01x02, J5 Conn_01x02, J6 Conn_01x02, J7 Conn_01x02, J8 Conn_01x02, J9 Conn_01x02, U1 STM32F446RETx, U10 MCP6001-OT, U11 MCP6001-OT, U3 DRV8833PWP_X, U4 DRV8833PWP_Y, U5 DRV8833PWP_Z, U6 MCP6001-OT, U7 MCP6001-OT, U8 MCP6001-OT, U9 MCP6001-OT

Commit message: ADCS: add input protection, ESD, decoupling and mounting holes
- PTC fuses, reverse-polarity P-MOSFETs and TVS diodes on 5V and 3.3V
- ESD diodes on sun-sensor inputs and I2C buses
- Bulk and local decoupling on 5V and 3.3V
- DRV8833 nFAULT pull-ups to 3.3V
- RC filters on current-sense ADC inputs, I2C pull-ups, BOOT0 pull-down
- Single 0R GND-GNDA tie
- Four 4 mm mounting holes
- Project footprint library for the Tag-Connect SWD footprint

DRC (KiCad 10.0.6): 0 violations, 0 unconnected pads.

Co-Authored-By: Claude Opus 5.5 <noreply@anthropic.com>
Parts:
- added C24: 47uF 10V, Capacitor_SMD:C_1206_3216Metric_Pad1.33x1.80mm_HandSolder, F.Cu at (137.9, 69.8)
- added C25: 10uF, Capacitor_SMD:C_0805_2012Metric_Pad1.18x1.45mm_HandSolder, F.Cu at (111.0, 58.6)
- added C26: 100nF, Capacitor_SMD:C_0805_2012Metric_Pad1.18x1.45mm_HandSolder, F.Cu at (138.4, 94.3)
- added C27: 100nF, Capacitor_SMD:C_0805_2012Metric_Pad1.18x1.45mm_HandSolder, F.Cu at (144.2, 96.8)
- added C28: 100nF, Capacitor_SMD:C_0805_2012Metric_Pad1.18x1.45mm_HandSolder, F.Cu at (152.7, 80.0)
- added C29: 100nF, Capacitor_SMD:C_0805_2012Metric_Pad1.18x1.45mm_HandSolder, F.Cu at (135.2, 77.1)
- added C30: 4.7uF, Capacitor_SMD:C_0805_2012Metric_Pad1.18x1.45mm_HandSolder, F.Cu at (134.7, 75.0)
- added C31: 100nF, Capacitor_SMD:C_0805_2012Metric_Pad1.18x1.45mm_HandSolder, F.Cu at (130.4, 84.5)
- added C32: 100nF, Capacitor_SMD:C_0805_2012Metric_Pad1.18x1.45mm_HandSolder, F.Cu at (132.5, 92.5)
- added C33: 100nF, Capacitor_SMD:C_0805_2012Metric_Pad1.18x1.45mm_HandSolder, F.Cu at (134.4, 94.7)
- added D1: SMBJ5.0A, Diode_SMD:D_SMB, F.Cu at (136.4, 66.2)
- added D10: ESD5B5, Diode_SMD:D_SOD-523, F.Cu at (138.8, 46.5)
- added D11: ESD5B5, Diode_SMD:D_SOD-523, F.Cu at (165.2, 53.6)
- added D12: ESD5B5, Diode_SMD:D_SOD-523, F.Cu at (169.9, 50.6)
- added D2: SMBJ3.3A, Diode_SMD:D_SMB, F.Cu at (114.3, 60.8)
- added D3: ESD5B5, Diode_SMD:D_SOD-523, F.Cu at (109.8, 84.8)
- added D4: ESD5B5, Diode_SMD:D_SOD-523, F.Cu at (119.2, 126.7)
- added D5: ESD5B5, Diode_SMD:D_SOD-523, F.Cu at (110.5, 100.2)
- added D6: ESD5B5, Diode_SMD:D_SOD-523, F.Cu at (102.8, 64.4)
- added D7: ESD5B5, Diode_SMD:D_SOD-523, F.Cu at (160.8, 125.1)
- added D8: ESD5B5, Diode_SMD:D_SOD-523, F.Cu at (170.1, 126.7)
- added D9: ESD5B5, Diode_SMD:D_SOD-523, F.Cu at (136.0, 46.5)
- added F1: 0.75A PTC, Fuse:Fuse_1206_3216Metric_Pad1.42x1.75mm_HandSolder, F.Cu at (126.5, 65.0)
- added F2: 0.5A PTC, Fuse:Fuse_1206_3216Metric_Pad1.42x1.75mm_HandSolder, F.Cu at (115.6, 54.6)
- added Q1: AO3401A, Package_TO_SOT_SMD:SOT-23, F.Cu at (130.7, 66.2)
- added Q2: AO3401A, Package_TO_SOT_SMD:SOT-23, F.Cu at (112.3, 54.6)
- added R12: 10k, Resistor_SMD:R_0805_2012Metric_Pad1.20x1.40mm_HandSolder, F.Cu at (141.9, 116.7)
- added R13: 10k, Resistor_SMD:R_0805_2012Metric_Pad1.20x1.40mm_HandSolder, F.Cu at (173.3, 95.8)
- added R14: 10k, Resistor_SMD:R_0805_2012Metric_Pad1.20x1.40mm_HandSolder, F.Cu at (174.6, 75.9)
- added R18: 10k, Resistor_SMD:R_0805_2012Metric_Pad1.20x1.40mm_HandSolder, F.Cu at (130.6, 69.0)
- added R19: 10k, Resistor_SMD:R_0805_2012Metric_Pad1.20x1.40mm_HandSolder, F.Cu at (108.5, 55.0)
- added R20: 0R, Resistor_SMD:R_0805_2012Metric_Pad1.20x1.40mm_HandSolder, F.Cu at (132.1, 88.8)
- added R21: 10k, Resistor_SMD:R_0805_2012Metric_Pad1.20x1.40mm_HandSolder, F.Cu at (139.0, 75.4)
- added R22: 4.7k, Resistor_SMD:R_0805_2012Metric_Pad1.20x1.40mm_HandSolder, F.Cu at (136.2, 56.1)
- added R23: 4.7k, Resistor_SMD:R_0805_2012Metric_Pad1.20x1.40mm_HandSolder, F.Cu at (142.2, 55.6)
- added R24: 1k, Resistor_SMD:R_0805_2012Metric_Pad1.20x1.40mm_HandSolder, F.Cu at (125.0, 85.5)
- added R25: 1k, Resistor_SMD:R_0805_2012Metric_Pad1.20x1.40mm_HandSolder, F.Cu at (125.7, 82.7)
- added R26: 1k, Resistor_SMD:R_0805_2012Metric_Pad1.20x1.40mm_HandSolder, F.Cu at (125.1, 90.1)
- C11, C6, C7: value 10uF -> 0.01uF
- C23: value 2.2uF -> 4.7uF
- renumbered REF** to H1, REF** to H2, REF** to H3, REF** to H4, R1_0805 to R15, R1_806 to R16, R1_807 to R17
Connections:
- net Net-(J4-Pin_1) renamed /SS1_IN
- net Net-(J5-Pin_1) renamed /SS2_IN
- net Net-(J6-Pin_1) renamed /SS3_IN
- net Net-(J7-Pin_1) renamed /SS4_IN
- net Net-(J8-Pin_1) renamed /SS5_IN
- net Net-(J9-Pin_1) renamed /SS6_IN
- J14 pad 1: /3.3V -> /3V3_IN
- J15 pad 1: /5V -> /5V_IN
- TP4 pad 1: /3.3V -> /3V3_IN
- TP5 pad 1: /5V -> /5V_IN
- U1 pad 10: unconnected-(U1-PC2-Pad10) -> /Z_AISEN_ADC
- U1 pad 60: GND -> /BOOT0
- U1 pad 8: unconnected-(U1-PC0-Pad8) -> /X_AISEN_ADC
- U1 pad 9: unconnected-(U1-PC1-Pad9) -> /Y_AISEN_ADC
Routing:
- net /3.3V: track 288.0 -> 390.3 mm, vias 6 -> 18
- net /X_AISEN: track 6.34 -> 92.4 mm, vias 0 -> 4
- net /Z_AISEN: track 9.69 -> 74.3 mm, vias 0 -> 6
- net GNDA: track 210.7 -> 273.8 mm, vias 8 -> 10
- net /Y_AISEN: track 14.0 -> 69.2 mm, vias 2 -> 7
- net /Y_AISEN_ADC: track 0.00 -> 50.8 mm, vias 0 -> 6
- net /Z_AISEN_ADC: track 0.00 -> 37.9 mm, vias 0 -> 6
- net GND: track 378.0 -> 413.7 mm, vias 5 -> 21
- net /X_AISEN_ADC: track 0.00 -> 25.0 mm, vias 0 -> 4
- net /3V3_IN: track 0.00 -> 18.6 mm, vias 0 -> 1
- net /5V_IN: track 0.00 -> 12.3 mm
- net /I2C1_SCL: track 33.6 -> 44.0 mm
- net /BOOT0: track 0.00 -> 10.0 mm, vias 0 -> 2
- net /5V_F: track 0.00 -> 9.29 mm, vias 0 -> 2
- net /5V: track 202.2 -> 194.1 mm
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