File: ADCS/ADCS.kicad_pcb (KiCad board)
At the start: 2 copper layers, 84 x 84 mm, 85 parts, among them J1 Conn_01x02, J10 Conn_01x04, J11 Conn_01x03, J12 Conn_01x08, J14 Conn_01x02, J15 Conn_01x02, J16 SWD_TagConnect, J2 Conn_01x02, J3 Conn_01x02, J4 Conn_01x02, J5 Conn_01x02, J6 Conn_01x02, J7 Conn_01x02, J8 Conn_01x02, J9 Conn_01x02, U1 STM32F446RETx, U10 MCP6001-OT, U11 MCP6001-OT, U3 DRV8833PWP_X, U4 DRV8833PWP_Y, U5 DRV8833PWP_Z, U6 MCP6001-OT, U7 MCP6001-OT, U8 MCP6001-OT, U9 MCP6001-OT

Commit message: Update ADCS PCB: review fixes (nFAULT, VCAP, I2C1 pull-ups, board size, decoupling)
- nFAULT: R12/R13/R14 (10k) now pull DRVX/Y/Z_FAULT up to 3.3V (were tied to GND,
  so the open-drain fault lines always read "fault")
- VCAP_1: C23 changed 2.2uF -> 4.7uF (LQFP-64 has a single VCAP pin; DS10693 Table 18)
- I2C1 (IMU bus): added R16/R17 4.7k pull-ups on I2C1_SCL/SDA
- Board: outline 84x84 -> 85x84 mm; mounting holes H1-H4 (4 mm) on a 74 x 76 mm
  pattern; dimensions moved off F.Cu onto User.Drawings
- Decoupling caps moved closer to the MCU pins: C27 0.6 mm, C24 1.8 mm,
  C25 2.5 mm (was 22.4), C22 3.1 mm, C26 4.7 mm, C21 5.2 mm, C28 5.9 mm
- PCB updated from schematic (no parity differences); DRC: 0 errors, 0 unconnected
Parts:
- added C24: 100nF, Capacitor_SMD:C_0603_1608Metric_Pad1.08x0.95mm_HandSolder, F.Cu at (138.9, 94.3)
- added C25: 100nF, Capacitor_SMD:C_0603_1608Metric_Pad1.08x0.95mm_HandSolder, F.Cu at (146.9, 93.9)
- added C26: 100nF, Capacitor_SMD:C_0603_1608Metric_Pad1.08x0.95mm_HandSolder, F.Cu at (151.7, 77.3)
- added C27: 100nF, Capacitor_SMD:C_0603_1608Metric_Pad1.08x0.95mm_HandSolder, F.Cu at (135.3, 79.3)
- added C28: 100nF, Capacitor_SMD:C_0603_1608Metric_Pad1.08x0.95mm_HandSolder, F.Cu at (133.1, 75.7)
- added C29: 4.7uF, Capacitor_SMD:C_0805_2012Metric_Pad1.18x1.45mm_HandSolder, F.Cu at (133.0, 77.5)
- added C30: 100nF, Capacitor_SMD:C_0603_1608Metric_Pad1.08x0.95mm_HandSolder, F.Cu at (116.0, 93.5)
- added C31: 100nF, Capacitor_SMD:C_0603_1608Metric_Pad1.08x0.95mm_HandSolder, F.Cu at (121.5, 110.0)
- added C32: 100nF, Capacitor_SMD:C_0603_1608Metric_Pad1.08x0.95mm_HandSolder, F.Cu at (117.0, 106.0)
- added C33: 100nF, Capacitor_SMD:C_0603_1608Metric_Pad1.08x0.95mm_HandSolder, F.Cu at (107.0, 77.4)
- added C34: 100nF, Capacitor_SMD:C_0603_1608Metric_Pad1.08x0.95mm_HandSolder, F.Cu at (151.0, 120.5)
- added C35: 100nF, Capacitor_SMD:C_0603_1608Metric_Pad1.08x0.95mm_HandSolder, F.Cu at (163.5, 109.6)
- added C36: 10uF, Capacitor_SMD:C_1206_3216Metric_Pad1.33x1.80mm_HandSolder, F.Cu at (113.4, 50.0)
- added C37: 10uF, Capacitor_SMD:C_1206_3216Metric_Pad1.33x1.80mm_HandSolder, F.Cu at (123.5, 67.0)
- added R12: 10k, Resistor_SMD:R_0805_2012Metric_Pad1.20x1.40mm_HandSolder, F.Cu at (153.5, 91.0)
- added R13: 10k, Resistor_SMD:R_0805_2012Metric_Pad1.20x1.40mm_HandSolder, F.Cu at (162.5, 91.5)
- added R14: 10k, Resistor_SMD:R_0805_2012Metric_Pad1.20x1.40mm_HandSolder, F.Cu at (164.0, 74.5)
- added R15: 0R, Resistor_SMD:R_0805_2012Metric_Pad1.20x1.40mm_HandSolder, F.Cu at (128.5, 108.0)
- added R16: 4.7k, Resistor_SMD:R_0805_2012Metric_Pad1.20x1.40mm_HandSolder, F.Cu at (135.5, 54.1)
- added R17: 4.7k, Resistor_SMD:R_0805_2012Metric_Pad1.20x1.40mm_HandSolder, F.Cu at (135.5, 56.3)
- C11, C6, C7: value 10uF -> 0.01uF
- C23: value 2.2uF -> 4.7uF
- J16: footprint Library:Tag-Connect_TC2030-IDC-NL_2x03_P1.27mm_Vertical -> Connector:Tag-Connect_TC2030-IDC-NL_2x03_P1.27mm_Vertical
- moved C22 9.76 mm to (130.9, 87.9)
- moved C21 3.65 mm to (128.9, 87.9)
- moved R2 2.50 mm to (127.7, 83.2)
- moved TP17 2.00 mm to (169.0, 110.2)
- moved H1 1.11 mm to (106.2, 49.0)
- moved H3 1.09 mm to (106.2, 125.0)
- moved H2 0.50 mm to (180.2, 49.0)
- moved H4 0.50 mm to (180.2, 125.0)
- moved TP13 0.25 mm to (116.0, 110.8)
- renumbered REF** to H1, REF** to H2, REF** to H3, REF** to H4
Routing:
- net /3.3V: track 288.0 -> 367.7 mm, vias 6 -> 11
- net GND: track 378.0 -> 430.1 mm, vias 5 -> 7
- net GNDA: track 210.7 -> 236.7 mm, vias 8 -> 7
- net /I2C1_SDA: track 31.7 -> 39.2 mm
- net /DRVZ_FAULT: track 31.8 -> 39.2 mm, vias 2 -> 3
- net /DRVY_FAULT: track 32.4 -> 39.0 mm
- net /I2C1_SCL: track 33.6 -> 38.2 mm
- net /DRVX_FAULT: track 31.5 -> 35.7 mm
- net /5V: track 202.2 -> 205.2 mm
- net /SS6: track 59.4 -> 60.9 mm
- net /SS1: track 42.0 -> 43.2 mm, vias 0 -> 2
- net Net-(U1-VCAP_1): track 8.44 -> 9.45 mm
- net /DRVZ_SLEEP: track 48.9 -> 49.9 mm, vias 2 -> 4
- net /DRVX_SLEEP: track 38.2 -> 38.9 mm
Other:
- board size 84 x 84 mm -> 85 x 84 mm
- board text removed: "ADCS SYSTEM Created by: PARTH S. KAKIRDE"

Commit message: Update ADCS and TTC KiCad designs
Routing:
- net /SS1: track 43.2 -> 42.5 mm
Other:
- board text added: "ADCS PCB 10/2026 VJTI Parth Kakirde Pushkar Dube Arpit Rajput"
