File: ADCS/ADCS.kicad_sch (KiCad schematic)
At the start: 84 parts, among them J1 Conn_01x02, J10 Conn_01x04, J11 Conn_01x03, J12 Conn_01x08, J14 Conn_01x02, J15 Conn_01x02, J16 SWD_TagConnect, J2 Conn_01x02, J3 Conn_01x02, J4 Conn_01x02, J5 Conn_01x02, J6 Conn_01x02, J7 Conn_01x02, J8 Conn_01x02, J9 Conn_01x02, U1 STM32F446RETx, U10 MCP6001-OT, U11 MCP6001-OT, U3 DRV8833PWP_X, U4 DRV8833PWP_Y, U5 DRV8833PWP_Z, U6 MCP6001-OT, U7 MCP6001-OT, U8 MCP6001-OT, U9 MCP6001-OT

Commit message: ADCS: add input protection, ESD, decoupling and mounting holes
- PTC fuses, reverse-polarity P-MOSFETs and TVS diodes on 5V and 3.3V
- ESD diodes on sun-sensor inputs and I2C buses
- Bulk and local decoupling on 5V and 3.3V
- DRV8833 nFAULT pull-ups to 3.3V
- RC filters on current-sense ADC inputs, I2C pull-ups, BOOT0 pull-down
- Single 0R GND-GNDA tie
- Four 4 mm mounting holes
- Project footprint library for the Tag-Connect SWD footprint

DRC (KiCad 10.0.6): 0 violations, 0 unconnected pads.

Co-Authored-By: Claude Opus 5.5 <noreply@anthropic.com>
Parts:
- added C24: 47uF 10V, Capacitor_SMD:C_1206_3216Metric_Pad1.33x1.80mm_HandSolder, symbol Device:C
- added C25: 10uF, Capacitor_SMD:C_0805_2012Metric_Pad1.18x1.45mm_HandSolder, symbol Device:C
- added C26, C27, C28, C29, C31, C32, C33: 100nF, Capacitor_SMD:C_0805_2012Metric_Pad1.18x1.45mm_HandSolder, symbol Device:C
- added C30: 4.7uF, Capacitor_SMD:C_0805_2012Metric_Pad1.18x1.45mm_HandSolder, symbol Device:C
- added D1: SMBJ5.0A, Diode_SMD:D_SMB, symbol Device:D_Zener
- added D10, D11, D12, D3, D4, D5, D6, D7, D8, D9: ESD5B5, Diode_SMD:D_SOD-523, symbol Device:D_TVS
- added D2: SMBJ3.3A, Diode_SMD:D_SMB, symbol Device:D_Zener
- added F1: 0.75A PTC, Fuse:Fuse_1206_3216Metric_Pad1.42x1.75mm_HandSolder, symbol Device:Polyfuse
- added F2: 0.5A PTC, Fuse:Fuse_1206_3216Metric_Pad1.42x1.75mm_HandSolder, symbol Device:Polyfuse
- added Q1, Q2: AO3401A, Package_TO_SOT_SMD:SOT-23, symbol Transistor_FET:AO3401A
- added R18, R19, R21: 10k, Resistor_SMD:R_0805_2012Metric_Pad1.20x1.40mm_HandSolder, symbol Device:R
- added R20: 0R, Resistor_SMD:R_0805_2012Metric_Pad1.20x1.40mm_HandSolder, symbol Device:R
- added R22, R23: 4.7k, Resistor_SMD:R_0805_2012Metric_Pad1.20x1.40mm_HandSolder, symbol Device:R
- added R24, R25, R26: 1k, Resistor_SMD:R_0805_2012Metric_Pad1.20x1.40mm_HandSolder, symbol Device:R
- C23: value 2.2uF -> 4.7uF
- renumbered R1_0805 to R15, R1_806 to R16, R1_807 to R17
Connections:
- net 3.3V: now also R12.2, R13.2, R14.1, C25.1, C26.1, C27.1, C28.1, C29.1, C30.1, D2.1 (K), Q2.2 (S), R22.1, R23.1; no longer J14.1 (Pin_1), TP4.1
- net 5V: now also C24.1, D1.1 (K), Q1.2 (S); no longer J15.1 (Pin_1), TP5.1
- net GND: now also C24.2, C25.2, C26.2, C27.2, C28.2, C29.2, C30.2, D1.2 (A), D10.2 (A2), D11.2 (A2), D12.2 (A2), D2.2 (A), D9.2 (A2), R18.2, R19.2, R20.2, R21.2; no longer R12.2, R13.2, R14.1, U1.60 (BOOT0)
- net GNDA: now also C31.2, C32.2, C33.2, D3.2 (A2), D4.2 (A2), D5.2 (A2), D6.2 (A2), D7.2 (A2), D8.2 (A2), R20.1
- net I2C1_SCL: now also D9.1 (A1), R22.2
- net I2C1_SDA: now also D10.1 (A1), R23.2
- net RPI_SCL: now also D11.1 (A1)
- net RPI_SDA: now also D12.1 (A1)
- net X_AISEN: now also R24.1
- net Y_AISEN: now also R25.1
- net Z_AISEN: now also R26.1
- net SS6_IN: now reaches C20.2, J9.1 (Pin_1), R9.2, U11.4 (-)
- net SS6_IN: now also D8.1 (A1)
- net SS5_IN: now reaches C19.2, J8.1 (Pin_1), R8.2, U10.4 (-)
- net SS5_IN: now also D7.1 (A1)
- net SS4_IN: now reaches C18.2, J7.1 (Pin_1), R7.2, U9.4 (-)
- net SS4_IN: now also D6.1 (A1)
- net SS1_IN: now reaches C15.2, J4.1 (Pin_1), R4.2, U6.4 (-)
- net SS1_IN: now also D3.1 (A1)
- net Z_AISEN_ADC: now reaches U1.10 (PC2)
- net Z_AISEN_ADC: now also C33.1, R26.2
- net X_AISEN_ADC: now reaches U1.8 (PC0)
- net X_AISEN_ADC: now also C31.1, R24.2
- net Y_AISEN_ADC: now reaches U1.9 (PC1)
- net Y_AISEN_ADC: now also C32.1, R25.2
- net SS2_IN: now reaches C16.2, J5.1 (Pin_1), R5.2, U7.4 (-)
- net SS2_IN: now also D4.1 (A1)
- net SS3_IN: now reaches C17.2, J6.1 (Pin_1), R6.2, U8.4 (-)
- net SS3_IN: now also D5.1 (A1)
- new net 3V3_F: F2.2, Q2.3 (D)
- new net 3V3_IN: F2.1, J14.1 (Pin_1), TP4.1
- new net 5V_F: F1.2, Q1.3 (D)
- new net 5V_IN: F1.1, J15.1 (Pin_1), TP5.1
- new net BOOT0: R21.1, U1.60 (BOOT0)
- new net Q1_G: Q1.1 (G), R18.1
- new net Q2_G: Q2.1 (G), R19.1
- no-connect marks 35 -> 32
Other:
- note added: "3.3V INPUT: J14 -> F2 -> Q2 (reverse polarity) -> 3.3V (D2 cathode on rail)"
- note added: "5V INPUT: J15 -> F1 -> Q1 (reverse polarity) -> 5V (D1 cathode on rail)"
- note added: "ADDED 2026-10-06: INPUT PROTECTION + PRE-FAB FIXES"
- note added: "BOOT0 PULL-DOWN + I2C1 PULL-UPS (IMU J12 / MAGNETOMETER J10)"
- note added: "COIL CURRENT TELEMETRY: AISEN (1 ohm sense) -> 1k/100nF -> PC0/PC1/PC2 (ADC123_IN10/11/12)"
- note added: "ESD ON OFF-BOARD LINES: sun sensors J4-J9 (to GNDA), I2C J10/J11/J12 (to GND)"
- note added: "STM32 VDD DECOUPLING (place one 100nF at each VDD pin 19/32/48/64) + GNDA-GND TIE (place R20 next to VSSA pin 12)"
