File: ADCS/ADCS.kicad_sch (KiCad schematic)
At the start: 84 parts, among them J1 Conn_01x02, J10 Conn_01x04, J11 Conn_01x03, J12 Conn_01x08, J14 Conn_01x02, J15 Conn_01x02, J16 SWD_TagConnect, J2 Conn_01x02, J3 Conn_01x02, J4 Conn_01x02, J5 Conn_01x02, J6 Conn_01x02, J7 Conn_01x02, J8 Conn_01x02, J9 Conn_01x02, U1 STM32F446RETx, U10 MCP6001-OT, U11 MCP6001-OT, U3 DRV8833PWP_X, U4 DRV8833PWP_Y, U5 DRV8833PWP_Z, U6 MCP6001-OT, U7 MCP6001-OT, U8 MCP6001-OT, U9 MCP6001-OT

Commit message: Update ADCS PCB: review fixes (nFAULT, VCAP, I2C1 pull-ups, board size, decoupling)
- nFAULT: R12/R13/R14 (10k) now pull DRVX/Y/Z_FAULT up to 3.3V (were tied to GND,
  so the open-drain fault lines always read "fault")
- VCAP_1: C23 changed 2.2uF -> 4.7uF (LQFP-64 has a single VCAP pin; DS10693 Table 18)
- I2C1 (IMU bus): added R16/R17 4.7k pull-ups on I2C1_SCL/SDA
- Board: outline 84x84 -> 85x84 mm; mounting holes H1-H4 (4 mm) on a 74 x 76 mm
  pattern; dimensions moved off F.Cu onto User.Drawings
- Decoupling caps moved closer to the MCU pins: C27 0.6 mm, C24 1.8 mm,
  C25 2.5 mm (was 22.4), C22 3.1 mm, C26 4.7 mm, C21 5.2 mm, C28 5.9 mm
- PCB updated from schematic (no parity differences); DRC: 0 errors, 0 unconnected
Parts:
- added C24, C25, C26, C27, C28, C30, C31, C32, C33, C34, C35: 100nF, Capacitor_SMD:C_0603_1608Metric_Pad1.08x0.95mm_HandSolder, symbol Device:C
- added C29: 4.7uF, Capacitor_SMD:C_0805_2012Metric_Pad1.18x1.45mm_HandSolder, symbol Device:C
- added C36, C37: 10uF, Capacitor_SMD:C_1206_3216Metric_Pad1.33x1.80mm_HandSolder, symbol Device:C
- added R15: 0R, Resistor_SMD:R_0805_2012Metric_Pad1.20x1.40mm_HandSolder, symbol Device:R
- added R16, R17: 4.7k, Resistor_SMD:R_0805_2012Metric_Pad1.20x1.40mm_HandSolder, symbol Device:R
- C23: value 2.2uF -> 4.7uF
- J16: footprint Library:Tag-Connect_TC2030-IDC-NL_2x03_P1.27mm_Vertical -> Connector:Tag-Connect_TC2030-IDC-NL_2x03_P1.27mm_Vertical
Connections:
- net 3.3V: now also R12.2, R13.2, R14.1, C24.1, C25.1, C26.1, C27.1, C28.1, C29.1, C30.1, C31.1, C32.1, C33.1, C34.1, C35.1, C36.1, R16.1, R17.1
- net 5V: now also C37.1
- net GND: now also C24.2, C25.2, C26.2, C27.2, C28.2, C29.2, C36.2, C37.2, R15.1; no longer R12.2, R13.2, R14.1
- net GNDA: now also C30.2, C31.2, C32.2, C33.2, C34.2, C35.2, R15.2
- net I2C1_SCL: now also R16.2
- net I2C1_SDA: now also R17.2
Other:
- note added: "Each cap < 2 mm from the pin written under it"
- note added: "GND-GNDA star point: place R15 at U1 VSSA (pin 12)"
- note added: "VBAT 1"
- note added: "VDD 19"
- note added: "VDD 32"
- note added: "VDD 48"
- note added: "VDD 64"
- note added: "VDDA 13"
- note added: "bulk"
- moved on the sheet: C15, C16, C17, C18, C19, C20, C21, C22, J4, J5, J6, J7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

Commit message: Update ADCS and TTC KiCad designs
Other:
- note removed: "Each cap < 2 mm from the pin written under it"
- note removed: "GND-GNDA star point: place R15 at U1 VSSA (pin 12)"
