File: EPS/CubeSat_EPS/CubeSat_EPS.kicad_pcb (KiCad board)
At the start: 2 copper layers, 85 x 84 mm, 46 parts, among them J1 SOLAR_IN, J10 AUX_POWER_OUT, J12 ADCS_5V_POWER, J13 ADCS_5V_POWER, J2 INA226_MODULE, J25 Pyro, J3 BMS_MODULE, J4 BATTERY_PACK, J6 OBC_INTERFACE, J8 ADCS_POWER, J9 TTC_POWER, Q1 P-MOSFET, Q3 IRLZ44N, U1 XL4015, U2 MP1584 Buck Converter, U3 CN3722_2S_MPPT_MODULE

Commit message: Update EPS PCB
Parts:
- moved H4 0.46 mm to (108.8, 129.9)
Other:
- board text added: "EPS PCB 10/2026 VJTI Abhijit Dalal Krish Sitafale"
