File: TTC/TTC_LoRa.kicad_pcb (KiCad board)
At the start: 2 copper layers, 85 x 84 mm, 81 parts, among them J1 EPS 3V3, J2 MISSION, J3 SMA edge, J4 SWD TC2030, J5 OBC I2C, J6 OBC UART, J7 EPS 5V, J8 SPARE GPIO, J9 DIPOLE FEED, Q1 AO3401A, U1 TPS7A2033PDBVR, U2 RFM98W-433S2, U3 STM32F446RET6, U4 TMP102, Y1 8MHz, Y2 32.768kHz

Commit message: TTC: pre-fab fixes - BURN_EN pull-down, NSS pull-up, crystal caps, I2C ESD
- R20 100k pull-down on BURN_EN (PC2), R21 10k pull-up on RFM_NSS
- C17/C18 12pF (HSE), C19/C20 8.2pF (LSE)
- D1 and D8 marked DNP (clamp voltages do not protect the rails)
- optional ESD diodes D9/D10 on OBC SDA/SCL
- J6 silkscreen TX/RX/G labels from the OBC side
KiCad ERC 0, DRC 0 (with schematic parity), 0 unconnected.

Co-Authored-By: Claude Sonnet 5.5 <noreply@anthropic.com>
Parts:
- added D10: ESD5B5, Diode_SMD:D_SOD-523, B.Cu at (139.4, 160.6)
- added D9: ESD5B5, Diode_SMD:D_SOD-523, B.Cu at (133.4, 158.0)
- added R20: 100k, Resistor_SMD:R_0603_1608Metric, F.Cu at (156.8, 141.8)
- added R21: 10k, Resistor_SMD:R_0603_1608Metric, B.Cu at (147.0, 141.8)
- C17, C18: value CL TBD -> 12pF
- C19, C20: value CL TBD -> 8.2pF
- D1: value SMBJ3.3A -> SMBJ3.3A DNP
- D8: value SMBJ5.0A -> SMBJ5.0A DNP
Routing:
- net /OBC_SCL: track 44.9 -> 47.1 mm
- net /OBC_SDA: track 31.8 -> 33.7 mm
- net +3V3: track 234.7 -> 235.9 mm
- net /RFM_NSS: track 46.3 -> 46.8 mm
Other:
- board text added: "G"
- board text added: "J6 OBC SIDE"
- board text added: "RX"
- board text added: "TX"
