File: TTC/TTC_LoRa.kicad_sch (KiCad schematic)
At the start: 74 parts, among them J1 EPS 3V3, J2 MISSION, J3 SMA edge, J4 SWD TC2030, J5 OBC I2C, J6 OBC UART, J7 EPS 5V, J8 SPARE GPIO, J9 DIPOLE FEED, Q1 AO3401A, U1 TPS7A2033PDBVR, U2 RFM98W-433S2, U3 STM32F446RET6, U4 TMP102, Y1 8MHz, Y2 32.768kHz

Commit message: TTC: pre-fab fixes - BURN_EN pull-down, NSS pull-up, crystal caps, I2C ESD
- R20 100k pull-down on BURN_EN (PC2), R21 10k pull-up on RFM_NSS
- C17/C18 12pF (HSE), C19/C20 8.2pF (LSE)
- D1 and D8 marked DNP (clamp voltages do not protect the rails)
- optional ESD diodes D9/D10 on OBC SDA/SCL
- J6 silkscreen TX/RX/G labels from the OBC side
KiCad ERC 0, DRC 0 (with schematic parity), 0 unconnected.

Co-Authored-By: Claude Sonnet 5.5 <noreply@anthropic.com>
Parts:
- added D10, D9: ESD5B5, Diode_SMD:D_SOD-523, symbol Device:D_TVS
- added R20: 100k, Resistor_SMD:R_0603_1608Metric, symbol Device:R
- added R21: 10k, Resistor_SMD:R_0603_1608Metric, symbol Device:R
- C17, C18: value CL TBD -> 12pF
- C19, C20: value CL TBD -> 8.2pF
- D1: value SMBJ3.3A -> SMBJ3.3A DNP; now not fitted
- D8: value SMBJ5.0A -> SMBJ5.0A DNP; now not fitted
Connections:
- net +3V3: now also R21.1
- net BURN_EN: now also R20.1
- net GND: now also D10.2 (A2), D9.2 (A2), R20.2
- net OBC_SCL: now also D10.1 (A1)
- net OBC_SDA: now also D9.1 (A1)
- net RFM_NSS: now also R21.2
Other:
- note added: "D9/D10: OBC I2C ESD (OPTIONAL). OBC board pull-ups sit in parallel with R11/R12"
- note added: "J6 (from OBC side): 1 = OBC TX to PA10 RX, 2 = OBC RX from PA9 TX, 3 = GND. Cross TX/RX is already done on the board"
- note added: "R20: BURN_EN PULL-DOWN"
- note added: "R21: NSS PULL-UP"
